File: kicad/udk_stm32g474_usb4_split.kicad_pcb (KiCad board)
At the start: 4 copper layers, 108.8 x 48 mm, 156 parts, among them J1 USB_A, J10 QWIIC, J11 ARGB, J12 5V, J13 USB_C_Receptacle, J14 Conn_01x08_Pin, J15 Conn_01x08_Pin, J16 TC2030-SWD, J17 Conn_01x02_Socket, J18 Conn_01x02_Socket, J2 USB_A, J5 USB_A, J8 SPI, J9 CONN, Q1 AO3401A, SW1 BOOT, SW2 RESET, U1 TS3USB30ERSWR, U10 REF3033E, U11 CH217K, U12 M25C-MEM-SPI, U13 TS3USB30ERSWR, U14 TS3USB30ERSWR, U15 TS3USB30ERSWR, U16 TS3USB30ERSWR, U17 LM66100DCK, U18 LM66100DCK, U19 LM66100DCK, U2 MCP23008-xML, U20 LP5907MFX-3.3, U21 NC7SZ125M5X, U22 LM66100DCK, U23 24AA02E48-OT, U3 CH334F, U4 LM66100DCK, U5 LM66100DCK, U6 STM32G474CBTx, U7 TS3USB30ERSWR, U8 LM66100DCK, U9 LM66100DCK, X1 Qwicc Logo, X2 Tecsmith Logo, X3 UDK Logo, X4 OSHW Logo, Y1 12MHz SMD3225-4P, Y2 8MHz SMD3225-4P

Commit message: added port esd
Parts:
- added C36: 4n7, Capacitor_SMD:C_0805_2012Metric_Pad1.18x1.45mm_HandSolder, F.Cu at (86.7, 84.5)
- added C37: 4n7, Capacitor_SMD:C_0805_2012Metric_Pad1.18x1.45mm_HandSolder, F.Cu at (167.3, 63.5)
- added R27: 1000K, Resistor_SMD:R_0805_2012Metric, F.Cu at (86.5, 82.5)
- added R28: 1000K, Resistor_SMD:R_0805_2012Metric, F.Cu at (167.5, 65.5)
- added Z2: SRV05-4, Package_SO:TSOP-6_1.65x3.05mm_P0.95mm, F.Cu at (149.5, 56.5)
- added Z3: SRV05-4, Package_SO:TSOP-6_1.65x3.05mm_P0.95mm, F.Cu at (89.8, 74.0)
- added Z4: SRV05-4, Package_SO:TSOP-6_1.65x3.05mm_P0.95mm, F.Cu at (164.0, 74.0)
- moved C27 8.73 mm to (167.6, 82.2), turned to 0 degrees
- moved C9 8.73 mm to (86.4, 65.8), turned to 180 degrees
- moved L4 0.45 mm to (180.2, 67.0)
- moved L8 0.45 mm to (180.2, 81.0)
Connections:
- net /U2x_D+ renamed U2x_D+
- net /U2x_D- renamed U2x_D-
Routing:
- net GND: track 276.8 -> 322.7 mm, vias 97 -> 105
- net U2x_D+: track 4.37 -> 20.0 mm
- net U2x_D-: track 4.50 -> 19.0 mm
- net U2_5V: track 10.6 -> 24.9 mm, vias 0 -> 2
- net U3_5V: track 34.2 -> 41.3 mm, vias 2 -> 4
- net U4_5V: track 49.3 -> 56.3 mm, vias 4 -> 6
- net LED4: track 201.9 -> 207.1 mm
- net (no net): track 3.38 -> 0.00 mm
- net GND_4: track 0.00 -> 3.26 mm
- net GND_3: track 0.00 -> 3.26 mm
- net ~{LED4}: track 57.4 -> 60.4 mm
- net 5V^{USB}: track 115.0 -> 117.8 mm
- net U4x_D-: track 26.1 -> 28.3 mm, vias 3 -> 2
- net U3x_D+: track 32.3 -> 32.0 mm, vias 4 -> 3
- net U4x_D+: track 22.8 -> 22.9 mm, vias 1 -> 0
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